Commit message: fixed names in urdfs

File: segwayrmp400_description/urdf/dual_em61_trailer.urdf.xacro (robot description, xacro)
@@ -1,4 +1,4 @@
 <?xml version="1.0"?>
-<robot xmlns:xacro="http://www.ros.org/wiki/xacro" name="atrv">
+<robot xmlns:xacro="http://www.ros.org/wiki/xacro" name="dual_em61_trailer">
 <!-- Some Color Materials -->
   <material name="Black"><color rgba="0.0 0.0 0.0 1.0"/></material>

File: segwayrmp400_description/urdf/segwayrmp400.urdf.xacro (robot description, xacro)
@@ -1,4 +1,4 @@
 <?xml version="1.0"?>
-<robot xmlns:xacro="http://www.ros.org/wiki/xacro" name="atrv">
+<robot xmlns:xacro="http://www.ros.org/wiki/xacro" name="segwayrmp400">
 <!-- Some Color Materials -->
   <material name="Green"><color rgba="0.0 0.8 0.0 1.0"/></material>
@@ -54,4 +54,11 @@
     </collision>
   </link>
+  <!-- hitch Link -->
+  <link name="hitch_link"/>
+  <joint name="base_hitch_joint" type="fixed">
+    <origin xyz="-0.56 0.0 0.0" rpy="0 0 0"/>
+    <parent link="base_link"/>
+    <child link="hitch_link"/>
+  </joint>
   <!-- This is a macro for the links that describe the wheels -->
   <xacro:macro name="wheel" params="prefix reflect_x reflect_y">
