Commit message: fixed bug in rviz files

File: segwayrmp400_description/urdf/segwayrmp400.urdf.xacro (robot description, xacro)
@@ -46,5 +46,5 @@
     <visual>
       <geometry>
-        <mesh filename="package://gavlab_atrv_description/meshes/atrv_chassis.dae"/>
+        <mesh filename="package://segwayrmp400_description/meshes/segwayrmp400.dae"/>
       </geometry>
       <!-- <material name="clear"/> -->
@@ -104,50 +104,3 @@
     <child link="imu_frame"/>
   </joint>
-  <!-- laser_link -->
-  <xacro:property name="laser_radius" value="0.045"/>
-  <xacro:property name="laser_height" value="0.16"/>
-  <link name="laser_link">
-    <xacro:default_inertial mass="3"/>
-    <visual>
-      <origin xyz="0 0 ${0.04-laser_height/2.0}" rpy="0 0 0"/>
-      <geometry>
-        <cylinder radius="${laser_radius}" length="${laser_height}"/>
-      </geometry>
-      <material name="Grey"/>
-    </visual>
-    <collision>
-      <origin xyz="0 0 ${0.04-laser_height/2.0}" rpy="0 0 0"/>
-      <geometry>
-        <cylinder radius="${laser_radius}" length="${laser_height}"/>
-      </geometry>
-    </collision>
-  </link>
-  <!-- base_link -> laser_link -->
-  <joint name="base_laser_joint" type="fixed">
-    <origin xyz="${0.015+laser_radius+chassis_length/2.0} 0 ${0.28-ground_clearance}" rpy="0 0 0"/>
-    <parent link="base_link"/>
-    <child link="laser_link"/>
-  </joint>
-  <!-- kinect_link -->
-  <link name="asus_link">
-    <xacro:default_inertial mass="0.0001"/>
-    <visual>
-      <origin xyz="0 0 0" rpy="0 0 0"/>
-      <geometry>
-        <mesh filename="package://gavlab_atrv_description/meshes/kinect.dae"/>
-      </geometry>
-    </visual>
-    <collision>
-      <origin xyz="0 0 0" rpy="0 0 0"/>
-      <geometry>
-        <box size="0.0730 0.2760 0.0720"/>
-      </geometry>
-    </collision>
-  </link>
-  <!-- base_link -> base_kinect_join -->
-  <joint name="base_kinect_joint" type="fixed">
-    <origin xyz="${(chassis_length/2)-0.19} 0 ${chassis_height+0.13-0.06}" rpy="0 0 0"/>
-    <parent link="base_link"/>
-    <child link="asus_link"/>
-  </joint>
 </robot>

Commit message: segway display working in rviz

File: segwayrmp400_description/urdf/segwayrmp400.urdf.xacro (robot description, xacro)
@@ -7,5 +7,5 @@
   <material name="Blue"><color rgba="0.0 0.0 0.8 1.0"/></material>
   <material name="Black"><color rgba="0.0 0.0 0.0 1.0"/></material>
-  <material name="Grey"><color rgba="0.7 0.7 0.7 0.7"/></material>
+  <material name="Grey"><color rgba="0.7 0.7 0.7 1.0"/></material>
   <material name="atrv_orange"><color rgba="0.8 0.16 0.0 1" /></material>
   <material name="clear"><color rgba="0 0 0 0"/></material>
@@ -45,8 +45,9 @@
     <xacro:default_inertial mass="80"/>
     <visual>
+      <origin xyz="0 0 0" rpy="0 0 0"/>
       <geometry>
-        <mesh filename="package://segwayrmp400_description/meshes/segwayrmp400.dae"/>
+        <mesh filename="package://segwayrmp400_description/meshes/segwayrmp400_chassis.stl"/>
       </geometry>
-      <!-- <material name="clear"/> -->
+      <material name="Grey"/>
     </visual>
     <collision>
@@ -70,7 +71,7 @@
         <origin xyz="0 0 ${wheel_width/2}" rpy="0 0 0" />
         <geometry>
-          <cylinder radius="${wheel_radius}" length="${wheel_width}"/>
+          <mesh filename="package://segwayrmp400_description/meshes/segwayrmp400_wheel.stl"/>
         </geometry>
-        <material name="Black"/>
+        <material name="Grey"/>
       </visual>
       <collision>
@@ -85,5 +86,5 @@
       <parent link="base_link"/>
       <child link="${prefix}_wheel_link"/>
-      <origin xyz="${(chassis_length/2 - wheel_radius)*reflect_x} ${(chassis_width/2 + 0.03)*reflect_y} ${wheel_radius - ground_clearance}"
+      <origin xyz="${(0.27)*reflect_x} ${(chassis_width/2 + 0.03)*reflect_y} ${0.1}"
               rpy="${(M_PI/2)*reflect_y*-1} 0 0"/>
     </joint>

Commit message: updating urdfs and meshes for em61 and segway

File: segwayrmp400_description/urdf/segwayrmp400.urdf.xacro (robot description, xacro)
@@ -7,5 +7,5 @@
   <material name="Blue"><color rgba="0.0 0.0 0.8 1.0"/></material>
   <material name="Black"><color rgba="0.0 0.0 0.0 1.0"/></material>
-  <material name="Grey"><color rgba="0.7 0.7 0.7 1.0"/></material>
+  <material name="Grey"><color rgba="0.3 0.3 0.3 1.0"/></material>
   <material name="atrv_orange"><color rgba="0.8 0.16 0.0 1" /></material>
   <material name="clear"><color rgba="0 0 0 0"/></material>
@@ -34,8 +34,4 @@
   </xacro:macro>
 <!-- links -->
-  <!-- base_footprint -->
-  <!-- The frame of the floor directly below the base_link and -->
-  <!-- is needed for the navigation stack to work properly -->
-  <link name="base_footprint"></link>
   <!-- base_link -->
   <!-- The link that is the origin of all of the components of the -->
@@ -58,10 +54,4 @@
     </collision>
   </link>
-  <!-- base_footprint -> base_link -->
-  <joint name="base_footprint_joint" type="fixed">
-      <origin xyz="0 0 ${ground_clearance}" rpy="0 0 0"/>
-      <parent link="base_footprint"/>
-      <child link="base_link"/>
-  </joint>
   <!-- This is a macro for the links that describe the wheels -->
   <xacro:macro name="wheel" params="prefix reflect_x reflect_y">
@@ -98,10 +88,3 @@
   <!-- right_rear_wheel_link -->
   <xacro:wheel prefix="right_rear" reflect_x="-1" reflect_y="-1" />
-  <!-- Imu Link -->
-  <link name="imu_frame"/>
-  <joint name="base_imu_joint" type="fixed">
-    <origin xyz="-0.11 0 0.27" rpy="0 0 0"/>
-    <parent link="base_link"/>
-    <child link="imu_frame"/>
-  </joint>
 </robot>

Commit message: added lidar link

File: segwayrmp400_description/urdf/segwayrmp400.urdf.xacro (robot description, xacro)
@@ -61,4 +61,11 @@
     <child link="hitch_link"/>
   </joint>
+  <!-- laser Link -->
+  <link name="base_laser_link"/>
+  <joint name="base_laser_joint" type="fixed">
+    <origin xyz="0.55 0.0 0.25" rpy="0 0 0"/>
+    <parent link="base_link"/>
+    <child link="base_laser_link"/>
+  </joint>
   <!-- This is a macro for the links that describe the wheels -->
   <xacro:macro name="wheel" params="prefix reflect_x reflect_y">
